Commit message: fixup! updated model

File: ros2_basics_ws/src/my_two_wheel_robot/model/MR_arm.urdf.xacro (robot description, xacro)
@@ -3,5 +3,6 @@
   <xacro:macro name="MR_arm" params="parent_link *joint_pose">
     <!-- Base link is the center of the robot's bottom plate -->
-    <joint name="MR_arm_joint" type="fixed">
+    <joint name="MR_arm_joint"
+      type="fixed">
       <parent link="${parent_link}" />
       <child link="link_0" />
@@ -32,4 +33,9 @@
     <!-- Joint 1 -->
     <link name="link_1">
+      <inertial>
+        <mass value="0.1" />
+        <origin xyz="0 0 0" rpy="0 0 0" />
+        <inertia ixx="0" ixy="0" ixz="0" iyy="0" iyz="0" izz="0" />
+      </inertial>
       <visual>
         <origin xyz="0 0 0" rpy="0 0 0" />
@@ -45,5 +51,6 @@
       </collision>
     </link>
-    <joint name="joint_shoulder" type="revolute">
+    <joint
+      name="joint_shoulder" type="revolute">
       <origin xyz="0 0 0.0575" rpy="0 0 0" />
       <parent link="link_1" />
@@ -54,4 +61,9 @@
     </joint>
     <link name="link_2">
+      <inertial>
+        <mass value="0.1" />
+        <origin xyz="0 0 0" rpy="0 0 0" />
+        <inertia ixx="0" ixy="0" ixz="0" iyy="0" iyz="0" izz="0" />
+      </inertial>
       <visual>
         <origin xyz="0 0 0" rpy="0 0 0" />
@@ -67,5 +79,6 @@
       </collision>
     </link>
-    <joint name="joint_elbow" type="revolute">
+    <joint
+      name="joint_elbow" type="revolute">
       <origin xyz="0 0 0.5" rpy="0 0 0" />
       <parent link="link_2" />
@@ -76,4 +89,9 @@
     </joint>
     <link name="link_3">
+      <inertial>
+        <mass value="0.1" />
+        <origin xyz="0 0 0" rpy="0 0 0" />
+        <inertia ixx="0" ixy="0" ixz="0" iyy="0" iyz="0" izz="0" />
+      </inertial>
       <visual>
         <origin xyz="0 0 0" rpy="0 0 0" />
@@ -89,5 +107,6 @@
       </collision>
     </link>
-    <joint name="joint_wrist_pitch" type="revolute">
+    <joint
+      name="joint_wrist_pitch" type="revolute">
       <origin xyz="0.4 0 0" rpy="0 0 0" />
       <parent link="link_3" />
@@ -98,4 +117,9 @@
     </joint>
     <link name="link_4">
+      <inertial>
+        <mass value="0.1" />
+        <origin xyz="0 0 0" rpy="0 0 0" />
+        <inertia ixx="0" ixy="0" ixz="0" iyy="0" iyz="0" izz="0" />
+      </inertial>
       <visual>
         <origin xyz="0 0 0" rpy="0 0 0" />
@@ -111,5 +135,6 @@
       </collision>
     </link>
-    <joint name="joint_wrist_roll" type="revolute">
+    <joint
+      name="joint_wrist_roll" type="revolute">
       <origin xyz="0.034 0 0" rpy="0 0 0" />
       <parent link="link_4" />
@@ -120,4 +145,9 @@
     </joint>
     <link name="link_5">
+      <inertial>
+        <mass value="0.1" />
+        <origin xyz="0 0 0" rpy="0 0 0" />
+        <inertia ixx="0" ixy="0" ixz="0" iyy="0" iyz="0" izz="0" />
+      </inertial>
       <visual>
         <origin xyz="0 0 0" rpy="0 0 0" />
@@ -133,5 +163,6 @@
       </collision>
     </link>
-    <joint name="joint_end_effector" type="revolute">
+    <joint
+      name="joint_end_effector" type="revolute">
       <origin xyz="0.050 -0.045 -0.01" rpy="0 0 1.570796327" />
       <parent link="link_5" />
@@ -150,4 +181,9 @@
     </joint>
     <link name="link_6">
+      <inertial>
+        <mass value="0.1" />
+        <origin xyz="0 0 0" rpy="0 0 0" />
+        <inertia ixx="0" ixy="0" ixz="0" iyy="0" iyz="0" izz="0" />
+      </inertial>
       <visual>
         <origin xyz="0 0 0" rpy="0 0 0" />
@@ -163,5 +199,11 @@
       </collision>
     </link>
-    <link name="link_7">
+    <link
+      name="link_7">
+      <inertial>
+        <mass value="0.1" />
+        <origin xyz="0 0 0" rpy="0 0 0" />
+        <inertia ixx="0" ixy="0" ixz="0" iyy="0" iyz="0" izz="0" />
+      </inertial>
       <visual>
         <origin xyz="0 0 0" rpy="0 0 0" />

File: ros2_basics_ws/src/my_two_wheel_robot/model/rover.urdf (robot description, URDF)
Before this commit: robot rover, 2 links, 1 joints
Links:
- removed link dummy_link
- added link chassis_link, mass 45.2; collision box size=0 0 0; visual mesh filename=file://$(find my_two_wheel_robot)/model/Full_Asm_Adjusted.d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
- link base_link: mass 45.2 -> None; geometry 
Joints:
- removed joint dummy_to_base
- added joint base_to_chassis: type fixed, parent base_link, child chassis_link, origin xyz=0 0 0.125

Commit message: rover sim working

File: ros2_basics_ws/src/my_two_wheel_robot/model/MR_arm.urdf.xacro (robot description, xacro)
@@ -13,11 +13,11 @@
         <origin xyz="0 0 0" rpy="0 0 0" />
         <geometry>
-          <mesh filename="package://my_two_wheel_robot/model/meshes/Link0.stl" />
-        </geometry>
-      </visual>
-      <collision>
-        <origin xyz="0 0 0" rpy="0 0 0" />
-        <geometry>
-          <mesh filename="package://my_two_wheel_robot/model/meshes/collision_Link0.stl" />
+          <mesh filename="file://$(find my_two_wheel_robot)/model/meshes/Link0.stl" />
+        </geometry>
+      </visual>
+      <collision>
+        <origin xyz="0 0 0" rpy="0 0 0" />
+        <geometry>
+          <mesh filename="file://$(find my_two_wheel_robot)/model/meshes/collision_Link0.stl" />
         </geometry>
       </collision>
@@ -41,11 +41,11 @@
         <origin xyz="0 0 0" rpy="0 0 0" />
         <geometry>
-          <mesh filename="package://my_two_wheel_robot/model/meshes/Link1.stl" />
-        </geometry>
-      </visual>
-      <collision>
-        <origin xyz="0 0 0" rpy="0 0 0" />
-        <geometry>
-          <mesh filename="package://my_two_wheel_robot/model/meshes/collision_Link1.stl" />
+          <mesh filename="file://$(find my_two_wheel_robot)/model/meshes/Link1.stl" />
+        </geometry>
+      </visual>
+      <collision>
+        <origin xyz="0 0 0" rpy="0 0 0" />
+        <geometry>
+          <mesh filename="file://$(find my_two_wheel_robot)/model/meshes/collision_Link1.stl" />
         </geometry>
       </collision>
@@ -69,11 +69,11 @@
         <origin xyz="0 0 0" rpy="0 0 0" />
         <geometry>
-          <mesh filename="package://my_two_wheel_robot/model/meshes/Link2.stl" />
-        </geometry>
-      </visual>
-      <collision>
-        <origin xyz="0 0 0" rpy="0 0 0" />
-        <geometry>
-          <mesh filename="package://my_two_wheel_robot/model/meshes/collision_Link2.stl" />
+          <mesh filename="file://$(find my_two_wheel_robot)/model/meshes/Link2.stl" />
+        </geometry>
+      </visual>
+      <collision>
+        <origin xyz="0 0 0" rpy="0 0 0" />
+        <geometry>
+          <mesh filename="file://$(find my_two_wheel_robot)/model/meshes/collision_Link2.stl" />
         </geometry>
       </collision>
@@ -97,11 +97,11 @@
         <origin xyz="0 0 0" rpy="0 0 0" />
         <geometry>
-          <mesh filename="package://my_two_wheel_robot/model/meshes/Link3.stl" />
-        </geometry>
-      </visual>
-      <collision>
-        <origin xyz="0 0 0" rpy="0 0 0" />
-        <geometry>
-          <mesh filename="package://my_two_wheel_robot/model/meshes/collision_Link3.stl" />
+          <mesh filename="file://$(find my_two_wheel_robot)/model/meshes/Link3.stl" />
+        </geometry>
+      </visual>
+      <collision>
+        <origin xyz="0 0 0" rpy="0 0 0" />
+        <geometry>
+          <mesh filename="file://$(find my_two_wheel_robot)/model/meshes/collision_Link3.stl" />
         </geometry>
       </collision>
@@ -125,11 +125,11 @@
         <origin xyz="0 0 0" rpy="0 0 0" />
         <geometry>
-          <mesh filename="package://my_two_wheel_robot/model/meshes/Link4.stl" />
-        </geometry>
-      </visual>
-      <collision>
-        <origin xyz="0 0 0" rpy="0 0 0" />
-        <geometry>
-          <mesh filename="package://my_two_wheel_robot/model/meshes/collision_Link4.stl" />
+          <mesh filename="file://$(find my_two_wheel_robot)/model/meshes/Link4.stl" />
+        </geometry>
+      </visual>
+      <collision>
+        <origin xyz="0 0 0" rpy="0 0 0" />
+        <geometry>
+          <mesh filename="file://$(find my_two_wheel_robot)/model/meshes/collision_Link4.stl" />
         </geometry>
       </collision>
@@ -153,11 +153,11 @@
         <origin xyz="0 0 0" rpy="0 0 0" />
         <geometry>
-          <mesh filename="package://my_two_wheel_robot/model/meshes/Link5.stl" />
-        </geometry>
-      </visual>
-      <collision>
-        <origin xyz="0 0 0" rpy="0 0 0" />
-        <geometry>
-          <mesh filename="package://my_two_wheel_robot/model/meshes/collision_Link5.stl" />
+          <mesh filename="file://$(find my_two_wheel_robot)/model/meshes/Link5.stl" />
+        </geometry>
+      </visual>
+      <collision>
+        <origin xyz="0 0 0" rpy="0 0 0" />
+        <geometry>
+          <mesh filename="file://$(find my_two_wheel_robot)/model/meshes/collision_Link5.stl" />
         </geometry>
       </collision>
@@ -189,5 +189,5 @@
         <origin xyz="0 0 0" rpy="0 0 0" />
         <geometry>
-          <mesh filename="package://my_two_wheel_robot/model/meshes/finger.stl" />
+          <mesh filename="file://$(find my_two_wheel_robot)/model/meshes/finger.stl" />
         </geometry>
       </visual>
@@ -209,5 +209,5 @@
         <origin xyz="0 0 0" rpy="0 0 0" />
         <geometry>
-          <mesh filename="package://my_two_wheel_robot/model/meshes/finger.stl" />
+          <mesh filename="file://$(find my_two_wheel_robot)/model/meshes/finger.stl" />
         </geometry>
       </visual>

File: ros2_basics_ws/src/my_two_wheel_robot/model/depth_camera.urdf.xacro (robot description, xacro)
@@ -17,5 +17,5 @@
                 <origin xyz="0 0 0" rpy="0 0 0" />
                 <geometry>
-                    <mesh filename="package://my_two_wheel_robot/model/meshes/depth_camera.dae"
+                    <mesh filename="file://$(find my_two_wheel_robot)/model/meshes/depth_camera.dae"
                         scale="1.0 1.0 1.0" />
                 </geometry>

File: ros2_basics_ws/src/my_two_wheel_robot/model/rover.urdf (robot description, URDF)
Before this commit: robot rover, 2 links, 1 joints
Links:
- link chassis_link: mass 45.2 -> ${chassis_mass}; geometry collision mesh filename=file://$(find my_two_wheel_robot)/model/meshes/Full_Asm_Adj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; visual mesh filename=file://$(find my_two_wheel_robot)/model/meshes/Full_Asm_Adj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

File: ros2_basics_ws/src/my_two_wheel_robot/model/rover.urdf.xacro (robot description, xacro)
@@ -1,25 +1,18 @@
-<?xml version="1.0"?>
 <robot xmlns:xacro="http://ros.org/wiki/xacro" name="rover">
+    <!-- Robot Parameters -->
+    <xacro:property name="chassis_mass" value="45.2" />
+    <!-- Part Includes - Payload, Sensors, Etc.. -->
     <xacro:include filename="$(find my_two_wheel_robot)/model/wheel.urdf.xacro" />
-    <!-- <xacro:include filename="$(find my_two_wheel_robot)/model/depth_camera.urdf.xacro" />a -->
-    <xacro:include filename="$(find my_two_wheel_robot)/model/MR_arm.urdf.xacro" />
+    <!-- <xacro:include filename="$(find my_two_wheel_robot)/model/depth_camera.urdf.xacro" />a
+    <xacro:include filename="$(find my_two_wheel_robot)/model/MR_arm.urdf.xacro" /> -->
+    <xacro:include filename="$(find my_two_wheel_robot)/model/imu.urdf" />
     <!-- Robot Definition -->
-    <link name="dummy_link" />
-    <joint name="dummy_to_base" type="fixed">
-        <parent link="dummy_link" />
-        <child link="base_link" />
-        <origin xyz="0 0 0" rpy="0 0 0" />
-    </joint>
-    <link name="base_link">
-        <inertial>
-            <origin xyz="0 0 0" rpy="0 0 0" />
-            <mass value="45.2" />
-            <!-- <inertia ixx="0" ixy="0.0" ixz="0.0" iyy="0" iyz="0.0" izz="0"/> -->
-            <inertia ixx="1.7724" ixy="0.0" ixz="0.0" iyy="0.141558" iyz="-0.0" izz="0.179826" />
-        </inertial>
+    <link name="base_link" />
+    <link name="chassis_link">
         <visual>
             <origin xyz="0 0 0.1" rpy="0 0 0" />
             <geometry>
-                <mesh filename="package://my_two_wheel_robot/model/meshes/Full_Asm_Adjusted.dae" />
+                <mesh
+                    filename="file://$(find my_two_wheel_robot)/model/meshes/Full_Asm_Adjusted.dae" />
             </geometry>
         </visual>
@@ -27,36 +20,56 @@
             <origin xyz="0 0 0.1" rpy="0 0 0" />
             <geometry>
-                <!-- <mesh
-                filename="package://my_two_wheel_robot/model/meshes/Full_Asm_Adjusted.dae"/> -->
-                <box size="0 0 0" />
+                <mesh
+                    filename="file://$(find my_two_wheel_robot)/model/meshes/Full_Asm_Adjusted.dae" />
+                <!-- <box size="0 0 0" /> -->
             </geometry>
         </collision>
+        <inertial>
+            <origin xyz="0 0 0" rpy="0 0 0" />
+            <mass value="${chassis_mass}" />
+            <!-- TODO FIXME The inertia below is invalid, using dummy 0 inertia -->
+            <!-- <inertia ixx="1.7724" ixy="0.0" ixz="0.0" iyy="0.141558" iyz="-0.0" izz="0.179826"
+            /> -->
+            <inertia ixx="0.0" ixy="0.0" ixz="0.0" iyy="0.0" iyz="0.0" izz="0.0" />
+        </inertial>
     </link>
-    <!-- <xacro:wheel wheel_prefix="left" parent_link="base_link">
-        <origin xyz="0.5125 -0.316275 ${-0.060752 + .1}" rpy="0 3.141592 0" />
+    <joint name="base_to_chassis" type="fixed">
+        <parent link="base_link" />
+        <child link="chassis_link" />
+        <origin xyz="0 0 0.125" />
+    </joint>
+    <!-- Wheels -->
+    <xacro:wheel wheel_prefix="lf" parent_link="base_link">
+        <origin xyz="0.5125 -0.316275 ${-0.060752 + .1}" rpy="0 1.57079 0" />
     </xacro:wheel>
-    <xacro:wheel wheel_prefix="right" parent_link="base_link">
-        <origin xyz="-0.5125 -0.316275 ${-0.060752 + .1}" rpy="0 0 0" />
+    <xacro:wheel wheel_prefix="rf" parent_link="base_link">
+        <origin xyz="-0.5125 -0.316275 ${-0.060752 + .1}" rpy="0 1.57079 0" />
     </xacro:wheel>
-    <xacro:wheel wheel_prefix="rear_left" parent_link="base_link">
-        <origin xyz="0.5125 0.306875 ${-0.060752 + .1}" rpy="0 3.141592 0" />
+    <xacro:wheel wheel_prefix="lb" parent_link="base_link">
+        <origin xyz="0.5125 0.306875 ${-0.060752 + .1}" rpy="0 1.57079 0" />
     </xacro:wheel>
-    <xacro:wheel wheel_prefix="rear_right" parent_link="base_link">
-        <origin xyz="-0.5125 0.306875 ${-0.060752 + .1}" rpy="0 0 0" />
-    </xacro:wheel> -->
-    <!-- <xacro:MR_arm parent_link="base_link">
+    <xacro:wheel wheel_prefix="rb" parent_link="base_link">
+        <origin xyz="-0.5125 0.306875 ${-0.060752 + .1}" rpy="0 1.57079 0" />
+    </xacro:wheel>
+    <!-- <xacro:depth_camera parent_link="base_link">
+        <origin xyz="0 -0.41 0.32" rpy="0 0 -1.57079" />
+    </xacro:depth_camera>
+    <xacro:MR_arm parent_link="base_link">
         <origin xyz="0 -0.28 0.37" rpy="0 0 -1.57079" />
     </xacro:MR_arm> -->
-    <!-- <xacro:depth_camera parent_link="base_link">
-        <origin xyz="0 0.2754 ${0.9943 + .1}" rpy="0 0 -1.57079" />
-    </xacro:depth_camera> -->
+    <!-- Gazebo Plugins -->
     <gazebo>
-        <plugin filename="libignition-gazebo-diff-drive-system.so"
-            name="ignition::gazebo::systems::DiffDrive">
-            <left_joint>left_wheel_joint</left_joint>
-            <right_joint>right_wheel_joint</right_joint>
+        <!-- Drive control -->
+        <plugin name="ignition::gazebo::systems::DiffDrive"
+            filename="ignition-gazebo-diff-drive-system">
+            <num_wheel_pairs>2</num_wheel_pairs>
+            <!-- Wheel Information -->
+            <left_joint>lf_wheel</left_joint>
+            <left_joint>rf_wheel</left_joint>
+            <right_joint>lb_wheel</right_joint>
+            <right_joint>rb_wheel</right_joint>
             <wheel_separation>0.63255</wheel_separation>
             <wheel_radius>0.1</wheel_radius>
-            <odom_publish_frequency>1</odom_publish_frequency>
+            <!-- Limits -->
             <max_linear_acceleration>1</max_linear_acceleration>
             <min_linear_acceleration>-1</min_linear_acceleration>
@@ -65,13 +78,28 @@
             <max_linear_velocity>0.5</max_linear_velocity>
             <min_linear_velocity>-0.5</min_linear_velocity>
-            <max_angular_velocity>1</max_angular_velocity>
-            <min_angular_velocity>-1</min_angular_velocity>
-            <topic>cmd_vel</topic>
+            <!-- Output -->
+            <frame_id>odom</frame_id>
+            <child_frame_id>base_link</child_frame_id>
+            <!-- Topics -->
+            <topic>/cmd_vel</topic>
+            <odom_topic>/odometry/wheels</odom_topic>
+            <tf_topic>/tf_gazebo</tf_topic>
         </plugin>
+        <plugin filename="ignition-gazebo-joint-state-publisher-system"
+            name="ignition::gazebo::systems::JointStatePublisher">
+            <topic>/joint_states</topic>
+        </plugin>
+        <!-- TODO FIXME doesn't work yet -->
+        <!-- IMU -->
+        <!-- <plugin filename="libignition-gazebo-imu-system" name="ignition::gazebo::systems::Imu"
+        />
+        <sensor name="imu" type="imu">
+            <always_on>1</always_on>
+            <update_rate>50</update_rate>
+            <visualize>true</visualize>
+            <topic>/imu/data</topic>
+            <enable_metrics>true</enable_metrics>
+            <ignition_frame_id>imu_link</ignition_frame_id>
+        </sensor> -->
     </gazebo>
-    <!-- <gazebo>
-        <plugin name="gazebo_ros_control" filename="libgazebo_ros_control.so">
-            <robotNamespace>/</robotNamespace>
-        </plugin>
-    </gazebo> -->
 </robot>

File: ros2_basics_ws/src/my_two_wheel_robot/model/wheel.urdf.xacro (robot description, xacro)
@@ -21,5 +21,5 @@
 				<geometry>
 					<mesh
-						filename="package://my_two_wheel_robot/model/meshes/full_wheel_assembly_fixed.dae" />
+						filename="file://$(find my_two_wheel_robot)/model/meshes/full_wheel_assembly_fixed.dae" />
 				</geometry>
 			</visual>

Commit message: renamed link for arm xacro

File: ros2_basics_ws/src/my_two_wheel_robot/model/MR_arm.urdf.xacro (robot description, xacro)
@@ -6,8 +6,8 @@
       type="fixed">
       <parent link="${parent_link}" />
-      <child link="link_0" />
+      <child link="link_0_base_waist" />
       <xacro:insert_block name="joint_pose" />
     </joint>
-    <link name="link_0">
+    <link name="link_0_base_waist">
       <visual>
         <origin xyz="0 0 0" rpy="0 0 0" />
@@ -25,6 +25,6 @@
     <joint name="joint_waist" type="revolute">
       <origin xyz="0 0 0" rpy="0 0 0" />
-      <parent link="link_0" />
-      <child link="link_1" />
+      <parent link="link_0_base_waist" />
+      <child link="link_1_waist_shoulder" />
       <axis xyz="0 0 1" />
       <limit effort="10.0" velocity="2.61799" lower="-3.141592" upper="3.141592" />
@@ -32,5 +32,5 @@
     </joint>
     <!-- Joint 1 -->
-    <link name="link_1">
+    <link name="link_1_waist_shoulder">
       <inertial>
         <mass value="0.1" />
@@ -54,11 +54,11 @@
       name="joint_shoulder" type="revolute">
       <origin xyz="0 0 0.0575" rpy="0 0 0" />
-      <parent link="link_1" />
-      <child link="link_2" />
+      <parent link="link_1_waist_shoulder" />
+      <child link="link_2_shoulder_elbow" />
       <axis xyz="0 1 0" />
       <limit effort="10.0" velocity="2.61799" lower="-1.570796327" upper="1.570796327" />
       <dynamics damping="0.5" />
     </joint>
-    <link name="link_2">
+    <link name="link_2_shoulder_elbow">
       <inertial>
         <mass value="0.1" />
@@ -82,11 +82,11 @@
       name="joint_elbow" type="revolute">
       <origin xyz="0 0 0.5" rpy="0 0 0" />
-      <parent link="link_2" />
-      <child link="link_3" />
+      <parent link="link_2_shoulder_elbow" />
+      <child link="link_3_elbow_wrist_pitch" />
       <axis xyz="0 1 0" />
       <limit effort="10.0" velocity="2.61799" lower="-1.570796327" upper="1.570796327" />
       <dynamics damping="0.5" />
     </joint>
-    <link name="link_3">
+    <link name="link_3_elbow_wrist_pitch">
       <inertial>
         <mass value="0.1" />
@@ -110,11 +110,11 @@
       name="joint_wrist_pitch" type="revolute">
       <origin xyz="0.4 0 0" rpy="0 0 0" />
-      <parent link="link_3" />
-      <child link="link_4" />
+      <parent link="link_3_elbow_wrist_pitch" />
+      <child link="link_4_wrist_pitch_wrist_roll" />
       <axis xyz="0 1 0" />
       <limit effort="10.0" velocity="2.61799" lower="-1.570796327" upper="1.570796327" />
       <dynamics damping="0.5" />
     </joint>
-    <link name="link_4">
+    <link name="link_4_wrist_pitch_wrist_roll">
       <inertial>
         <mass value="0.1" />
@@ -138,11 +138,11 @@
       name="joint_wrist_roll" type="revolute">
       <origin xyz="0.034 0 0" rpy="0 0 0" />
-      <parent link="link_4" />
-      <child link="link_5" />
+      <parent link="link_4_wrist_pitch_wrist_roll" />
+      <child link="link_5_wrist_roll_end_effector" />
       <axis xyz="1 0 0" />
       <limit effort="10.0" velocity="2.61799" lower="-3.141592" upper="3.141592" />
       <dynamics damping="0.5" />
     </joint>
-    <link name="link_5">
+    <link name="link_5_wrist_roll_end_effector">
       <inertial>
         <mass value="0.1" />
@@ -166,6 +166,6 @@
       name="joint_end_effector" type="revolute">
       <origin xyz="0.050 -0.045 -0.01" rpy="0 0 1.570796327" />
-      <parent link="link_5" />
-      <child link="link_6" />
+      <parent link="link_5_wrist_roll_end_effector" />
+      <child link="link_6_end_effector_1" />
       <axis xyz="0 0 1" />
       <limit effort="10.0" velocity="2.61799" lower="-3.141592" upper="3.141592" />
@@ -174,11 +174,11 @@
     <joint name="joint_7" type="revolute">
       <origin xyz="0.050 0.045 -0.01" rpy="0 3.141592 1.570796327" />
-      <parent link="link_5" />
-      <child link="link_7" />
+      <parent link="link_5_wrist_roll_end_effector" />
+      <child link="link_7_end_effector_2" />
       <axis xyz="0 0 1" />
       <limit effort="10.0" velocity="2.61799" lower="-3.141592" upper="3.141592" />
       <dynamics damping="0.5" />
     </joint>
-    <link name="link_6">
+    <link name="link_6_end_effector_1">
       <inertial>
         <mass value="0.1" />
@@ -200,5 +200,5 @@
     </link>
     <link
-      name="link_7">
+      name="link_7_end_effector_2">
       <inertial>
         <mass value="0.1" />
